File: botz-nxp.kicad_pcb (KiCad board)
At the start: 2 copper layers, 1 part

Commit message: Init
Parts:
- removed REF**: DFN-8-1EP_3x3mm_P0.65mm_EP1.55x2.4mm, Package_DFN_QFN:DFN-8-1EP_3x3mm_P0.65mm_EP1.55x2.4mm
- added C1: 0.1uF, PCM_SparkFun-Capacitor:C_0402_1005Metric, F.Cu at (163.2, 102.9)
- added C2: 0.1uF, PCM_SparkFun-Capacitor:C_0402_1005Metric, F.Cu at (163.2, 104.9)
- added C3: 0.1uF, PCM_SparkFun-Capacitor:C_0402_1005Metric, F.Cu at (163.2, 106.9)
- added C4: 0.1uF, PCM_SparkFun-Capacitor:C_0402_1005Metric, F.Cu at (163.2, 108.8)
- added C5: 4.7uF, PCM_SparkFun-Capacitor:C_0402_1005Metric, F.Cu at (163.2, 110.8)
- added C6: 0.1uF, PCM_SparkFun-Capacitor:C_0402_1005Metric, F.Cu at (163.2, 112.8)
- added D3: Red, PCM_SparkFun-LED:LED_0402_1005Metric_Red, F.Cu at (163.6, 130.4)
- added D4: PESD3V3L4UG, PCM_SparkFun-Semiconductor-Standard:SOT-353, F.Cu at (160.2, 131.4)
- added F1: 6V/0.5A/1A, PCM_SparkFun-Fuse:0805, F.Cu at (160.4, 134.5)
- added IC1: MCXA265VLH, Package_QFP:LQFP-64_10x10mm_P0.5mm, F.Cu at (154.6, 109.2)
- added J1: microSD, PCM_SparkFun-Connector:microSD_External_Pin, F.Cu at (138.4, 113.9)
- added J2: JST_1mm_4, PCM_SparkFun-Connector:JST_1x04_P1.0mm_Horizontal_SMD, F.Cu at (151.4, 117.7)
- added J3: Conn_01x04_Pin, PCM_SparkFun-Connector:JST_1x04_P1.0mm_Horizontal_SMD, F.Cu at (151.4, 124.5)
- added J5: JST_1mm_4, PCM_SparkFun-Connector:JST_1x04_P1.0mm_Horizontal_SMD, F.Cu at (151.4, 131.3)
- added J6: Conn_01x06_FPC_1.0mm, PCM_SparkFun-Connector:FPC_1x05_P1.0mm_Horizontal_DualContact_LIF, F.Cu at (160.3, 121.2)
- added J7: Conn_01x12, PCM_SparkFun-Connector:JST_1x12_P1.0mm_Horizontal_SMD, F.Cu at (137.4, 132.5)
- added L1: 120 Ohm, PCM_SparkFun-Capacitor:C_0603_1608Metric, F.Cu at (160.4, 137.1)
- added R1: 10k, PCM_SparkFun-Resistor:R_0402_1005Metric, F.Cu at (157.0, 130.4)
- added R6: 10k, PCM_SparkFun-Resistor:R_0402_1005Metric, F.Cu at (157.0, 132.4)
- added R7: 10k, PCM_SparkFun-Resistor:R_0402_1005Metric, F.Cu at (157.0, 134.4)
- added R8: 150, PCM_SparkFun-Resistor:R_0402_1005Metric, F.Cu at (157.0, 136.4)
Other:
- copper layers 2 -> 4
