File: botz-nxp.kicad_sch (KiCad schematic)
At the start: 12 parts, among them IC1 MCXA265VLH, J1 microSD, J2 JST_1mm_4, U2 MCP2561-E-MF, U3 MCP2561-E-MF

Commit message: Init
Parts:
- removed U2, U3: MCP2561-E-MF, Package_DFN_QFN:DFN-8-1EP_3x3mm_P0.65mm_EP1.55x2.4mm, symbol Interface_CAN_LIN:MCP2561-E-MF
- added D3: Red, PCM_SparkFun-LED:LED_0402_1005Metric_Red, symbol PCM_SparkFun-LED:LED_Red_0402
- added D4: PESD3V3L4UG, PCM_SparkFun-Semiconductor-Standard:SOT-353, symbol PCM_SparkFun-DiscreteSemi:D_TVS_ESD_4_3.3V
- added F1: 6V/0.5A/1A, PCM_SparkFun-Fuse:0805, symbol PCM_SparkFun-Fuse:Fuse 6V/0.5A/1A
- added J3: Conn_01x04_Pin, PCM_SparkFun-Connector:JST_1x04_P1.0mm_Horizontal_SMD, symbol Connector:Conn_01x04_Pin
- added J5: JST_1mm_4, PCM_SparkFun-Connector:JST_1x04_P1.0mm_Horizontal_SMD, symbol PCM_SparkFun-Connector:Conn_01x04_JST_P1.0mm_Horizontal_SMD
- added J6: Conn_01x06_FPC_1.0mm, PCM_SparkFun-Connector:FPC_1x05_P1.0mm_Horizontal_DualContact_LIF, symbol PCM_SparkFun-Connector:Conn_01x06_FPC_P1.0mm_Horizontal_DualContact_LIF
- added J7: Conn_01x12, PCM_SparkFun-Connector:JST_1x12_P1.0mm_Horizontal_SMD, symbol PCM_SparkFun-Connector:Conn_01x12_JST_P1.0mm_Horizontal_SMD
- added R1, R6, R7: 10k, PCM_SparkFun-Resistor:R_0402_1005Metric, symbol PCM_SparkFun-Resistor:10k_0402
- added R8: 150, PCM_SparkFun-Resistor:R_0402_1005Metric, symbol PCM_SparkFun-Resistor:150_0402
- IC1: footprint QFP50P1200X1200X160-64N -> Package_QFP:LQFP-64_10x10mm_P0.5mm
Connections:
- net 3.3V: now also J1.4 (VDD), D4.5 (K4), F1.1, J3.4 (Pin_4), R1.2, R6.1; no longer J2.1
- net GND: now also J1.10 (SHIELD), J1.6 (VSS), D3.1 (K), D4.2 (A), J3.3 (Pin_3), J6.3 (Pin_3), R7.1; no longer J2.2
- net J_RX: now also IC1.20 (P2_6), J6.5 (Pin_5); no longer J2.4
- net J_TX: now also IC1.21 (P2_7), J6.4 (Pin_4); no longer J2.3
- net CS1: now reaches J1.2 (DAT3/CD)
- net CS1: now also IC1.44 (P3_6), R6.2
- net SD01: now reaches J1.3 (CMD/SDI)
- net SD01: now also IC1.23 (P2_13)
- net SCK1: now reaches J1.5 (CLK/SCK)
- net SCK1: now also IC1.22 (P2_12)
- net SDI1: now reaches J1.7 (DAT0/SDO)
- net SDI1: now also IC1.24 (P2_15)
- net DET: now reaches J1.9 (~{DET})
- net DET: now also IC1.43 (P3_7)
- net RXD0: now reaches IC1.14 (P2_0)
- net RXD0: now also J2.3
- net TXD0: now reaches IC1.15 (P2_1)
- net TXD0: now also J2.4
- net DAC0_OUT: now reaches IC1.16 (P2_2)
- net DAC0_OUT: now also J7.12 (Pin_12)
- net IRQ: now reaches IC1.18 (P2_4)
- net CS2: now reaches IC1.19 (P2_5)
- net RXD1: now reaches IC1.2 (P1_8)
- net RXD1: now also J2.1
- net at IC1.25 (VDD_USB): now also R7.2
- net TXD1: now reaches IC1.3 (P1_9)
- net TXD1: now also J2.2
- net PWM1_B0: now reaches IC1.30 (P3_31)
- net PWM1_B0: now also J7.1 (Pin_1)
- net PWM1_A0: now reaches IC1.31 (P3_30)
- net PWM1_A0: now also J7.2 (Pin_2)
- net LORA_RST: now reaches IC1.32 (P3_29)
- net PWM1_B3: now reaches IC1.33 (P3_28)
- net PWM1_B3: now also J7.3 (Pin_3)
- net PWM1_A3: now reaches IC1.34 (P3_27)
- net PWM1_A3: now also J7.4 (Pin_4)
- net PWM1_B1: now reaches IC1.35 (P3_15)
- net PWM1_B1: now also J7.5 (Pin_5)
- net PWM1_A1: now reaches IC1.36 (P3_14)
- net PWM1_A1: now also J7.6 (Pin_6)
- net PWM1_B2: now reaches IC1.37 (P3_13)
- net PWM1_B2: now also J7.7 (Pin_7)
- net PWM1_A2: now reaches IC1.38 (P3_12)
- net PWM1_A2: now also J7.8 (Pin_8)
- net PWM0_B2: now reaches IC1.39 (P3_11)
- net PWM0_B2: now also J7.9 (Pin_9)
- net CAN0_TXD: now reaches IC1.4 (P1_10)
- net PWM0_A2: now reaches IC1.40 (P3_10)
- net PWM0_A2: now also J7.10 (Pin_10)
- net PWM0_B1: now reaches IC1.41 (P3_9)
- net PWM0_B1: now also J7.11 (Pin_11)
- net SWDIO: now reaches IC1.49 (P0_0)
- net SWDIO: now also J3.1 (Pin_1)
- net CAN0_RXD: now reaches IC1.5 (P1_11)
- net SWCLK: now reaches IC1.50 (P0_1)
- net SWCLK: now also J3.2 (Pin_2)
- net SWO: now reaches IC1.51 (P0_2)
- net SD02: now reaches IC1.56 (P1_0)
- net SCK2: now reaches IC1.57 (P1_1)
- net SDI2: now reaches IC1.58 (P1_2)
- net CAN1_RXD: now reaches IC1.6 (P1_12)
- net CAN1_TXD: now reaches IC1.7 (P1_13)
- net RST: now reaches IC1.8 (P1_29)
- net RST: now also J6.6 (Pin_6), R1.1
- net at IC1.9 (P1_30): now also R8.2
- new net: D3.2 (A), R8.1
- new net: F1.2, J6.2 (Pin_2)
- new net 5V: D4.4 (K3), J6.1 (Pin_1)
- new net CAN0H: J5.1
- new net CAN0L: J5.2
- new net CAN1H: J5.3
- new net CAN1L: J5.4
- no-connect marks 0 -> 2
Other:
- moved on the sheet: C1, C2, C3, C4, C5, C6, IC1, J1, L1
